File: PCB/focus-totem.kicad_pcb (KiCad board)
At the start: 2 copper layers, 84 x 72 mm, 17 parts, among them J1 SSD1306_0.91, SW1 SW_Push, SW2 SW_Push, SW3 SW_Push, SW4 EC11, U1 XIAO-RP2040

Commit message: Update to files and images
Other:
- board text added: "FOCUS TOTEM"
